File: hardware/hardware.kicad_pcb (KiCad board)
At the start: 2 copper layers, 53 x 38 mm, 13 parts, among them J1 Screw_Terminal_01x06, J2 ISP, U1 ATtiny25-20SSU

Commit message: things changed
Parts:
- moved C3 21.5 mm to (104.5, 130.5), turned to 180 degrees
Routing:
- net POT: track 27.4 -> 25.0 mm
- net GND: vias 2 -> 7
